File: LM2596_buck_5/LM2596_buck_5.kicad_pcb (KiCad board)
At the start: 2 copper layers, 65 x 30 mm, 7 parts, among them J1 Input, J2 Output, U1 LM2596T-5

Commit message: design  improvements
Parts:
- moved D1 10.0 mm to (121.6, 93.0)
- moved J1 8.60 mm to (104.0, 104.5), turned to 90 degrees
- moved J2 8.11 mm to (158.0, 103.5), turned to 90 degrees
- moved U1 6.00 mm to (127.6, 104.7)
Routing:
- net GND: track 82.2 -> 0.00 mm
- net VCC: track 28.7 -> 23.7 mm
- net Net-(C2-Pad1): track 34.3 -> 31.3 mm
- net Net-(D1-Pad1): track 29.1 -> 31.8 mm
- added copper zone on F.Cu, net GND
Other:
- board size 65 x 30 mm -> 67 x 33 mm
- board text added: "LM2596 5V Buck Regulator"
